File: kicad files/single radio pcb.kicad_pcb (KiCad board)
At the start: 4 copper layers, 37.7 x 37.7 mm, 56 parts, among them J1 Conn_Coaxial, J10 Conn_01x01_Female, J11 Conn_01x01_Female, J3 Conn_01x01_Female, J4 Conn_01x01_Female, J5 Conn_01x01_Female, J6 Conn_01x01_Female, J7 Conn_01x04_Male, J8 Conn_Coaxial, U1 3V3. 500mA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

Commit message: Updates including dif filter by antenna, better WiFi PCB antenna, and single inductor
Parts:
- removed U5: 2450FM07D0034T, Anyleaf Shared:2450FM07D0034
- added C14: 1.2p, Capacitor_SMD:C_0402_1005Metric, F.Cu at (149.8, 113.0)
- added C15: 1.2p, Capacitor_SMD:C_0402_1005Metric, F.Cu at (148.8, 114.2)
- added C16: 1.2p, Capacitor_SMD:C_0402_1005Metric, F.Cu at (150.8, 113.0)
- added C20: 1.2p, Capacitor_SMD:C_0402_1005Metric, F.Cu at (143.0, 115.2)
- added L2: 3n, Inductor_SMD:L_0402_1005Metric, F.Cu at (148.2, 112.5)
- added L3: 3n, Inductor_SMD:L_0402_1005Metric, F.Cu at (147.8, 114.2)
- Y2: value 52Mhz, 12pF -> 52Mhz, 8pF
- moved U4 6.16 mm to (142.1, 112.4), turned to -90 degrees
- moved R4 2.61 mm to (148.7, 116.3), turned to 90 degrees
- moved C4 1.27 mm to (134.7, 114.2)
- moved C6 1.27 mm to (134.8, 113.2)
- moved C7 1.27 mm to (137.5, 116.0)
- moved L1 1.27 mm to (136.8, 117.5)
- moved U2 1.27 mm to (138.7, 112.5)
- moved Y2 1.27 mm to (134.5, 111.2)
- moved R3 0.75 mm to (150.3, 114.5), turned to 180 degrees
- moved U6 0.50 mm to (145.0, 112.0)
- moved C3 0.25 mm to (137.8, 109.0)
- moved C5 0.25 mm to (139.8, 109.0)
Connections:
- J1 pad 1: Net-(J1-Pad1) -> Net-(C16-Pad1)
- U2 pad 22: /RF_OUT -> /RADIO_OUT
- U4 pad 1: /ANT1 -> /RADIO_OUT
- U4 pad 3: Net-(J1-Pad1) -> /FRONTEND_IN
- U6 pad 6: /RF_OUT -> /FRONTEND_IN
Routing:
- net /ANT_TRACE: track 4.56 -> 31.3 mm
- net GND: track 36.5 -> 44.9 mm
- net Net-(R3-Pad2): track 12.1 -> 16.9 mm
- net Net-(C16-Pad1): track 0.00 -> 3.75 mm
- net /BUSY: track 22.1 -> 18.4 mm
- net Net-(R4-Pad1): track 10.8 -> 14.3 mm
- net Net-(R3-Pad1): track 9.05 -> 12.4 mm
- net Net-(C20-Pad1): track 1.85 -> 4.86 mm
- net /ANT1: track 1.24 -> 3.90 mm
- net /RF_OUT: track 1.80 -> 0.00 mm
- net /RADIO_OUT: track 0.00 -> 1.70 mm
- net /FRONTEND_IN: track 0.00 -> 1.53 mm
- net Net-(J1-Pad1): track 1.32 -> 0.00 mm
- net /ANT2: track 1.28 -> 2.54 mm
- net /RST: track 18.3 -> 19.2 mm
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