File: kicad files/single radio schematic.kicad_sch (KiCad schematic)
At the start: 44 parts, among them J1 Conn_Coaxial, J10 Conn_01x01_Female, J11 Conn_01x01_Female, J3 Conn_01x01_Female, J4 Conn_01x01_Female, J5 Conn_01x01_Female, J6 Conn_01x01_Female, J7 Conn_01x04_Male, J8 Conn_Coaxial, U1 3V3. 500mA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

Commit message: Updates including dif filter by antenna, better WiFi PCB antenna, and single inductor
Parts:
- removed U5: 2450FM07D0034T, Anyleaf_Shared:2450FM07D0034, symbol Anyleaf Shared:2450FM07D0034
- added C14, C15, C16, C20: 1.2p, Capacitor_SMD:C_0402_1005Metric, symbol Device:C
- added L2, L3: 3n, Inductor_SMD:L_0402_1005Metric, symbol Device:L
- U2: LCSC C2151551 -> C125969
- Y2: value 52Mhz, 12pF -> 52Mhz, 8pF; LCSC (none) -> C781783; LCSC Seikio Epson (none) -> C841202; Mouser (none) -> 729-FW520WFMT1
Connections:
- net ANT1: now also C14.1, L2.1; no longer U4.1
- net ANT2: now also C15.1, L3.1
- net GND: now also C14.2, C15.2, C16.2, C20.2
- net at J1.1 (In): now also C16.1, L2.2; no longer U4.3
- net at J8.1 (In): now also C20.1, L3.2
- net RF_OUT renamed FRONTEND_IN
- net FRONTEND_IN: now also U4.3; no longer U2.22 (RFIO)
- new net RADIO_OUT: U2.22 (RFIO), U4.1
Other:
- note added: "3v3 regulator, since some FCs don't have a 3v3 line. Also, an ELRS spec requirement."
- note added: "Filter IC between the radio and frontend. These single-ICs are specifically designed for the SX1280, and save board space compared to a multi-part filter."
- note added: "Pi filters between frontend and antennas"
- note added: "WiFi PCB trace antenna. Wavelength = 125mm. 1/4 wavelength = 31.25mm A detailed doc on 2.4Ghz antenna traces: https://www.ti.com/lit/an/swra117d/swra117d.pdf Phil's Lab video on designing a PCB trace antenna: https://www.youtube.com/watch?v=yxU_Kw2de08 We've ommitted hte matching filter network and ideal shape due to low space availability, and WiFi not being part of this device's primary functio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"
- note removed: "3v3 regulator, since some FCs don't have a 3v3 line. Also, an ELRS team requirement."
- note removed: "Filter ICs between the RF frontend and antennas. These single-ICs are specifically designed for the SX1280, and save board space compared to a multi-part filter."
- moved on the sheet: C17, C18, C19, C3, C5, C6, C7, J1, J8, R1, R3, R4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
